Commit message: rviz partially done

File: src/simple_box_robo/model/robot.urdf.xacro (robot description, xacro)
@@ -20,5 +20,4 @@
   <!-- PI constant -->
   <xacro:property name="PI" value="3.141592" />
-  <xacro:property name="pi" value="${PI}" /> <!-- Alias for compatibility -->
   <!-- Material Color -->
   <material name="red">
@@ -57,4 +56,12 @@
     </inertial>
   </xacro:macro>
+  <!-- Add this at the top of your URDF, before base_link -->
+  <link name="dummy">
+  </link>
+  <joint name="dummy_joint" type="fixed">
+    <parent link="dummy"/>
+    <child link="base_link"/>
+  </joint>
+<!-- Keep your existing base_link and other elements -->
   <!-- ========== MAIN BODY ========== -->
   <link name="base_link">
@@ -93,11 +100,11 @@
       </geometry>
       <material name="almost_blue" />
-      <origin xyz="0 0 0" rpy="${pi/2} 0 0" />
-    </visual>
-    <collision>
-      <geometry>
-        <cylinder length="${wheel_len}" radius="${wheel_radius}" />
-      </geometry>
-      <origin xyz="0 0 0" rpy="${pi/2} 0 0" />
+      <origin xyz="0 0 0" rpy="${PI/2} 0 0" />
+    </visual>
+    <collision>
+      <geometry>
+        <cylinder length="${wheel_len}" radius="${wheel_radius}" />
+      </geometry>
+      <origin xyz="0 0 0" rpy="${PI/2} 0 0" />
     </collision>
     <xacro:inertia_wheel />
@@ -116,11 +123,11 @@
       </geometry>
       <material name="almost_blue" />
-      <origin xyz="0 0 0" rpy="${pi/2} 0 0" />
-    </visual>
-    <collision>
-      <geometry>
-        <cylinder length="${wheel_len}" radius="${wheel_radius}" />
-      </geometry>
-      <origin xyz="0 0 0" rpy="${pi/2} 0 0" />
+      <origin xyz="0 0 0" rpy="${PI/2} 0 0" />
+    </visual>
+    <collision>
+      <geometry>
+        <cylinder length="${wheel_len}" radius="${wheel_radius}" />
+      </geometry>
+      <origin xyz="0 0 0" rpy="${PI/2} 0 0" />
     </collision>
     <xacro:inertia_wheel />
@@ -139,11 +146,11 @@
       </geometry>
       <material name="almost_blue" />
-      <origin xyz="0 0 0" rpy="${pi/2} 0 0" />
-    </visual>
-    <collision>
-      <geometry>
-        <cylinder length="${wheel_len}" radius="${wheel_radius}" />
-      </geometry>
-      <origin xyz="0 0 0" rpy="${pi/2} 0 0" />
+      <origin xyz="0 0 0" rpy="${PI/2} 0 0" />
+    </visual>
+    <collision>
+      <geometry>
+        <cylinder length="${wheel_len}" radius="${wheel_radius}" />
+      </geometry>
+      <origin xyz="0 0 0" rpy="${PI/2} 0 0" />
     </collision>
     <xacro:inertia_wheel />
@@ -162,11 +169,11 @@
       </geometry>
       <material name="almost_blue" />
-      <origin xyz="0 0 0" rpy="${pi/2} 0 0" />
-    </visual>
-    <collision>
-      <geometry>
-        <cylinder length="${wheel_len}" radius="${wheel_radius}" />
-      </geometry>
-      <origin xyz="0 0 0" rpy="${pi/2} 0 0" />
+      <origin xyz="0 0 0" rpy="${PI/2} 0 0" />
+    </visual>
+    <collision>
+      <geometry>
+        <cylinder length="${wheel_len}" radius="${wheel_radius}" />
+      </geometry>
+      <origin xyz="0 0 0" rpy="${PI/2} 0 0" />
     </collision>
     <xacro:inertia_wheel />
