Commit message: Robo Started Moving

File: src/simple_box_robo/model/robot.gazebo.xacro (robot description, xacro)
@@ -1,6 +1,23 @@
 <?xml version="1.0"?>
 <robot xmlns:xacro="http://ros.org/wiki/xacro" name="simple_box_bot_gazebo">
-  <!-- ========== GAZEBO EXTENSIONS ========== -->
-  <!-- Required sensors system plugin -->
+  <!-- ROS 2 Control -->
+  <ros2_control name="diff_drive_controller" type="system">
+    <hardware>
+      <plugin>gz_ros2_control/GazeboSystem</plugin>
+    </hardware>
+    <joint name="body_to_lf_wheel">
+      <command_interface name="velocity"/>
+    </joint>
+    <joint name="body_to_lb_wheel">
+      <command_interface name="velocity"/>
+    </joint>
+    <joint name="body_to_rf_wheel">
+      <command_interface name="velocity"/>
+    </joint>
+    <joint name="body_to_rb_wheel">
+      <command_interface name="velocity"/>
+    </joint>
+  </ros2_control>
+  <!-- Gazebo Plugins -->
   <gazebo>
     <plugin filename="libignition-gazebo-sensors-system.so" name="ignition::gazebo::systems::Sensors">
@@ -8,5 +25,5 @@
     </plugin>
   </gazebo>
-  <!-- Differential Drive Plugin (unchanged, already correct) -->
+  <!-- Differential Drive Plugin (FIXED CONFIG) -->
   <gazebo>
     <plugin filename="libignition-gazebo-diff-drive-system.so" name="ignition::gazebo::systems::DiffDrive">
@@ -18,5 +35,5 @@
       <wheel_radius>${wheel_radius}</wheel_radius>
       <odom_publish_frequency>50</odom_publish_frequency>
-      <topic>cmd_vel</topic>
+      <topic>/model/simple_box_robo/cmd_vel</topic>  <!-- ABSOLUTE TOPIC -->
       <odom_topic>odom</odom_topic>
       <odom_frame>odom</odom_frame>
@@ -24,5 +41,5 @@
     </plugin>
   </gazebo>
-  <!-- GPU LIDAR (updated for Ignition Gazebo) -->
+  <!-- GPU LIDAR -->
   <gazebo reference="lidar_body">
     <sensor name="gpu_lidar" type="gpu_lidar">
@@ -45,13 +62,7 @@
           <resolution>0.01</resolution>
         </range>
-        <noise>
-          <type>gaussian</type>
-          <mean>0.0</mean>
-          <stddev>0.01</stddev>
-        </noise>
       </ray>
-      <plugin
-        filename="libignition-gazebo-gpu-lidar-system.so"
-        name="ignition::gazebo::systems::GpuLidar">
+      <plugin filename="libignition-gazebo-gpu-lidar-system.so"
+              name="ignition::gazebo::systems::GpuLidar">
         <topic>scan</topic>
         <frame_name>lidar_body</frame_name>
@@ -59,5 +70,5 @@
     </sensor>
   </gazebo>
-  <!-- Camera (updated plugin syntax) -->
+  <!-- Camera -->
   <gazebo reference="camera_link">
     <sensor name="camera_sensor" type="camera">
@@ -68,5 +79,4 @@
           <width>640</width>
           <height>480</height>
-          <format>R8G8B8</format>
         </image>
         <clip>
@@ -74,13 +84,7 @@
           <far>100</far>
         </clip>
-        <noise>
-          <type>gaussian</type>
-          <mean>0.0</mean>
-          <stddev>0.007</stddev>
-        </noise>
       </camera>
-      <plugin
-        filename="libignition-gazebo-camera-system.so"
-        name="ignition::gazebo::systems::Camera">
+      <plugin filename="libignition-gazebo-camera-system.so"
+              name="ignition::gazebo::systems::Camera">
         <topic>camera/image</topic>
         <frame_name>camera_link</frame_name>
@@ -88,24 +92,23 @@
     </sensor>
   </gazebo>
-  <!-- Gazebo materials (unchanged) -->
-  <gazebo reference="base_link">
-    <material>Gazebo/Green</material>
+  <!-- Wheel Physics (CRITICAL ADDITION) -->
+  <gazebo reference="rf_wheel">
+    <mu1 value="1.0"/>
+    <mu2 value="1.0"/>
+    <material>Gazebo/Blue</material>
   </gazebo>
-  <gazebo reference="rod">
-    <material>Gazebo/White</material>
-  </gazebo>
-  <gazebo reference="lidar_body">
-    <material>Gazebo/Red</material>
-  </gazebo>
-  <gazebo reference="rf_wheel">
+  <gazebo reference="lf_wheel">
+    <mu1 value="1.0"/>
+    <mu2 value="1.0"/>
     <material>Gazebo/Blue</material>
   </gazebo>
   <gazebo reference="rb_wheel">
-    <material>Gazebo/Blue</material>
-  </gazebo>
-  <gazebo reference="lf_wheel">
+    <mu1 value="1.0"/>
+    <mu2 value="1.0"/>
     <material>Gazebo/Blue</material>
   </gazebo>
   <gazebo reference="lb_wheel">
+    <mu1 value="1.0"/>
+    <mu2 value="1.0"/>
     <material>Gazebo/Blue</material>
   </gazebo>

File: src/simple_box_robo/model/robot.urdf.xacro (robot description, xacro)
@@ -1,4 +1,6 @@
 <?xml version="1.0"?>
 <robot xmlns:xacro="http://ros.org/wiki/xacro" name="simple_box_bot">
+  <!-- Add ROS 2 Control Import -->
+  <xacro:include filename="ros2_control.urdf.xacro" />
   <!-- ========== PROPERTIES ========== -->
   <!-- Dimension of the body -->
@@ -56,4 +58,6 @@
     </inertial>
   </xacro:macro>
+  <!-- ROS 2 Control Configuration (replace existing block) -->
+  <xacro:ros2_control name="diff_drive_controller" prefix="" />
   <!-- Add this at the top of your URDF, before base_link -->
   <link name="dummy">

Commit message: Differential Movement reeady

File: src/simple_box_robo/model/robot.gazebo.xacro (robot description, xacro)
@@ -1,29 +1,5 @@
 <?xml version="1.0"?>
 <robot xmlns:xacro="http://ros.org/wiki/xacro" name="simple_box_bot_gazebo">
-  <!-- ROS 2 Control -->
-  <ros2_control name="diff_drive_controller" type="system">
-    <hardware>
-      <plugin>gz_ros2_control/GazeboSystem</plugin>
-    </hardware>
-    <joint name="body_to_lf_wheel">
-      <command_interface name="velocity"/>
-    </joint>
-    <joint name="body_to_lb_wheel">
-      <command_interface name="velocity"/>
-    </joint>
-    <joint name="body_to_rf_wheel">
-      <command_interface name="velocity"/>
-    </joint>
-    <joint name="body_to_rb_wheel">
-      <command_interface name="velocity"/>
-    </joint>
-  </ros2_control>
-  <!-- Gazebo Plugins -->
-  <gazebo>
-    <plugin filename="libignition-gazebo-sensors-system.so" name="ignition::gazebo::systems::Sensors">
-      <render_engine>ogre2</render_engine>
-    </plugin>
-  </gazebo>
-  <!-- Differential Drive Plugin (FIXED CONFIG) -->
+  <!-- Differential Drive Plugin -->
   <gazebo>
     <plugin filename="libignition-gazebo-diff-drive-system.so" name="ignition::gazebo::systems::DiffDrive">
@@ -35,5 +11,5 @@
       <wheel_radius>${wheel_radius}</wheel_radius>
       <odom_publish_frequency>50</odom_publish_frequency>
-      <topic>/model/simple_box_robo/cmd_vel</topic>  <!-- ABSOLUTE TOPIC -->
+      <topic>cmd_vel</topic>
       <odom_topic>odom</odom_topic>
       <odom_frame>odom</odom_frame>
@@ -41,56 +17,58 @@
     </plugin>
   </gazebo>
-  <!-- GPU LIDAR -->
-  <gazebo reference="lidar_body">
-    <sensor name="gpu_lidar" type="gpu_lidar">
-      <pose>0 0 0 0 0 0</pose>
-      <visualize>false</visualize>
-      <update_rate>10</update_rate>
-      <topic>scan</topic>
-      <ray>
-        <scan>
-          <horizontal>
-            <samples>360</samples>
-            <resolution>1</resolution>
-            <min_angle>0</min_angle>
-            <max_angle>6.28319</max_angle>
-          </horizontal>
-        </scan>
-        <range>
-          <min>0.10</min>
-          <max>10.0</max>
-          <resolution>0.01</resolution>
-        </range>
-      </ray>
-      <plugin filename="libignition-gazebo-gpu-lidar-system.so"
-              name="ignition::gazebo::systems::GpuLidar">
-        <topic>scan</topic>
-        <frame_name>lidar_body</frame_name>
-      </plugin>
-    </sensor>
+  <!-- Keyboard Control Plugins -->
+  <gazebo>
+    <!-- Forward (Up Arrow) -->
+    <plugin filename="libignition-gazebo-triggered-publisher-system.so"
+            name="ignition::gazebo::systems::TriggeredPublisher">
+      <input type="ignition.msgs.Int32" topic="/keyboard/keypress">
+        <match field="data">16777235</match>
+      </input>
+      <output type="ignition.msgs.Twist" topic="/cmd_vel">
+        linear: {x: 0.5}, angular: {z: 0.0}
+      </output>
+    </plugin>
+    <!-- Backward (Down Arrow) -->
+    <plugin filename="libignition-gazebo-triggered-publisher-system.so"
+            name="ignition::gazebo::systems::TriggeredPublisher">
+      <input type="ignition.msgs.Int32" topic="/keyboard/keypress">
+        <match field="data">16777237</match>
+      </input>
+      <output type="ignition.msgs.Twist" topic="/cmd_vel">
+        linear: {x: -0.5}, angular: {z: 0.0}
+      </output>
+    </plugin>
+    <!-- Left (Left Arrow) -->
+    <plugin filename="libignition-gazebo-triggered-publisher-system.so"
+            name="ignition::gazebo::systems::TriggeredPublisher">
+      <input type="ignition.msgs.Int32" topic="/keyboard/keypress">
+        <match field="data">16777234</match>
+      </input>
+      <output type="ignition.msgs.Twist" topic="/cmd_vel">
+        linear: {x: 0.0}, angular: {z: 1.0}
+      </output>
+    </plugin>
+    <!-- Right (Right Arrow) -->
+    <plugin filename="libignition-gazebo-triggered-publisher-system.so"
+            name="ignition::gazebo::systems::TriggeredPublisher">
+      <input type="ignition.msgs.Int32" topic="/keyboard/keypress">
+        <match field="data">16777236</match>
+      </input>
+      <output type="ignition.msgs.Twist" topic="/cmd_vel">
+        linear: {x: 0.0}, angular: {z: -1.0}
+      </output>
+    </plugin>
+    <!-- Stop Signal (S)-->
+    <plugin filename="libignition-gazebo-triggered-publisher-system.so"
+            name="ignition::gazebo::systems::TriggeredPublisher">
+      <input type="ignition.msgs.Int32" topic="/keyboard/keypress">
+        <match field="data">83</match>
+      </input>
+      <output type="ignition.msgs.Twist" topic="/cmd_vel">
+        linear: {x: 0.0}, angular: {z: 0.0}
+      </output>
+    </plugin>
   </gazebo>
-  <!-- Camera -->
-  <gazebo reference="camera_link">
-    <sensor name="camera_sensor" type="camera">
-      <pose>0 0 0 0 0 0</pose>
-      <camera name="camera">
-        <horizontal_fov>1.0472</horizontal_fov>
-        <image>
-          <width>640</width>
-          <height>480</height>
-        </image>
-        <clip>
-          <near>0.1</near>
-          <far>100</far>
-        </clip>
-      </camera>
-      <plugin filename="libignition-gazebo-camera-system.so"
-              name="ignition::gazebo::systems::Camera">
-        <topic>camera/image</topic>
-        <frame_name>camera_link</frame_name>
-      </plugin>
-    </sensor>
-  </gazebo>
-  <!-- Wheel Physics (CRITICAL ADDITION) -->
+  <!-- Wheel Physics -->
   <gazebo reference="rf_wheel">
     <mu1 value="1.0"/>

File: src/simple_box_robo/model/robot.urdf.xacro (robot description, xacro)
@@ -2,5 +2,4 @@
 <robot xmlns:xacro="http://ros.org/wiki/xacro" name="simple_box_bot">
   <!-- Add ROS 2 Control Import -->
-  <xacro:include filename="ros2_control.urdf.xacro" />
   <!-- ========== PROPERTIES ========== -->
   <!-- Dimension of the body -->
@@ -58,6 +57,4 @@
     </inertial>
   </xacro:macro>
-  <!-- ROS 2 Control Configuration (replace existing block) -->
-  <xacro:ros2_control name="diff_drive_controller" prefix="" />
   <!-- Add this at the top of your URDF, before base_link -->
   <link name="dummy">
@@ -117,5 +114,5 @@
     <parent link="base_link" />
     <child link="rf_wheel" />
-    <origin xyz="${body_x/2 - 1.2*wheel_radius} ${-body_y/2 + wheel_len} ${wheel_z}" rpy="0 0 0" />
+    <origin xyz="${body_x/2 - 1.2*wheel_radius} ${-body_y/2} ${wheel_z}" rpy="0 0 0" />
     <axis xyz="0 1 0" />
   </joint>
@@ -140,5 +137,5 @@
     <parent link="base_link" />
     <child link="rb_wheel" />
-    <origin xyz="${-body_x/2 + 1.2*wheel_radius} ${-body_y/2 + wheel_len} ${wheel_z}" rpy="0 0 0" />
+    <origin xyz="${-body_x/2 + 1.2*wheel_radius} ${-body_y/2} ${wheel_z}" rpy="0 0 0" />
     <axis xyz="0 1 0" />
   </joint>
@@ -163,5 +160,5 @@
     <parent link="base_link" />
     <child link="lf_wheel" />
-    <origin xyz="${body_x/2 - 1.2*wheel_radius} ${body_y/2 - wheel_len} ${wheel_z}" rpy="0 0 0" />
+    <origin xyz="${body_x/2 - 1.2*wheel_radius} ${body_y/2} ${wheel_z}" rpy="0 0 0" />
     <axis xyz="0 1 0" />
   </joint>
@@ -186,5 +183,5 @@
     <parent link="base_link" />
     <child link="lb_wheel" />
-    <origin xyz="${-body_x/2 + 1.2*wheel_radius} ${body_y/2 - wheel_len} ${wheel_z}" rpy="0 0 0" />
+    <origin xyz="${-body_x/2 + 1.2*wheel_radius} ${body_y/2} ${wheel_z}" rpy="0 0 0" />
     <axis xyz="0 1 0" />
   </joint>
@@ -216,10 +213,9 @@
     </inertial>
   </link>
-  <joint name="body_to_rod" type="prismatic">
+  <joint name="body_to_rod" type="fixed">
     <parent link="base_link" />
     <child link="rod" />
     <origin xyz="${body_x/2 - lidar_x} 0 ${body_z + wheel_radius}" rpy="0 0 0" />
     <axis xyz="0 0 1" />
-    <limit lower="${body_z + wheel_radius}" upper="${body_z + wheel_radius + rod_z/2}" effort="10.0" velocity="1.0" />
   </joint>
   <!-- Lidar Main Body -->

Commit message: Lidar is working..

File: src/simple_box_robo/model/robot.gazebo.xacro (robot description, xacro)
@@ -1,4 +1,9 @@
 <?xml version="1.0"?>
 <robot xmlns:xacro="http://ros.org/wiki/xacro" name="simple_box_bot_gazebo">
+  <!-- Sensors System Plugin (MUST be top-level) -->
+  <!-- Joint State Publisher -->
+  <plugin filename="libignition-gazebo-joint-state-publisher-system.so"
+          name="ignition::gazebo::systems::JointStatePublisher">
+  </plugin>
   <!-- Differential Drive Plugin -->
   <gazebo>
@@ -46,5 +51,5 @@
       </input>
       <output type="ignition.msgs.Twist" topic="/cmd_vel">
-        linear: {x: 0.0}, angular: {z: 1.0}
+        linear: {x: 0.0}, angular: {z: 1.5}
       </output>
     </plugin>
@@ -56,5 +61,5 @@
       </input>
       <output type="ignition.msgs.Twist" topic="/cmd_vel">
-        linear: {x: 0.0}, angular: {z: -1.0}
+        linear: {x: 0.0}, angular: {z: -1.5}
       </output>
     </plugin>
@@ -69,4 +74,40 @@
       </output>
     </plugin>
+  </gazebo>
+  <!-- ROS-Ignition Bridge for LiDAR -->
+  <!-- LiDAR Sensor -->
+  <gazebo reference="lidar_body">
+    <sensor name="lidar_sensor" type="gpu_lidar">
+      <pose>0 0 0 0 0 0</pose>
+      <topic>lidar</topic>
+      <update_rate>10</update_rate>
+      <ray>
+        <scan>
+          <horizontal>
+            <samples>640</samples>
+            <resolution>1</resolution>
+            <min_angle>-1.396263</min_angle>  <!-- ~-80° -->
+            <max_angle>1.396263</max_angle>    <!-- ~80° -->
+          </horizontal>
+          <vertical>
+            <samples>1</samples>
+            <resolution>0.01</resolution>
+            <min_angle>0</min_angle>
+            <max_angle>0</max_angle>
+          </vertical>
+        </scan>
+        <range>
+          <min>0.08</min>
+          <max>10.0</max>
+          <resolution>0.01</resolution>
+        </range>
+      </ray>
+      <always_on>true</always_on>
+      <visualize>true</visualize>
+      <plugin filename="libignition-gazebo-sensors-system.so"
+          name="ignition::gazebo::systems::Sensors">
+        <render_engine>ogre2</render_engine>
+      </plugin>
+    </sensor>
   </gazebo>
   <!-- Wheel Physics -->

File: src/simple_box_robo/model/robot.urdf.xacro (robot description, xacro)
@@ -217,5 +217,4 @@
     <child link="rod" />
     <origin xyz="${body_x/2 - lidar_x} 0 ${body_z + wheel_radius}" rpy="0 0 0" />
-    <axis xyz="0 0 1" />
   </joint>
   <!-- Lidar Main Body -->

Commit message: Camera and Obstacle node is working with some issue

File: src/simple_box_robo/model/robot.gazebo.xacro (robot description, xacro)
@@ -30,5 +30,5 @@
         <match field="data">16777235</match>
       </input>
-      <output type="ignition.msgs.Twist" topic="/cmd_vel">
+      <output type="ignition.msgs.Twist" topic="/keyboard_cmd">
         linear: {x: 0.5}, angular: {z: 0.0}
       </output>
@@ -40,5 +40,5 @@
         <match field="data">16777237</match>
       </input>
-      <output type="ignition.msgs.Twist" topic="/cmd_vel">
+      <output type="ignition.msgs.Twist" topic="/keyboard_cmd">
         linear: {x: -0.5}, angular: {z: 0.0}
       </output>
@@ -50,6 +50,6 @@
         <match field="data">16777234</match>
       </input>
-      <output type="ignition.msgs.Twist" topic="/cmd_vel">
-        linear: {x: 0.0}, angular: {z: 1.5}
+      <output type="ignition.msgs.Twist" topic="/keyboard_cmd">
+        linear: {x: 0.0}, angular: {z: 2.5}
       </output>
     </plugin>
@@ -60,6 +60,6 @@
         <match field="data">16777236</match>
       </input>
-      <output type="ignition.msgs.Twist" topic="/cmd_vel">
-        linear: {x: 0.0}, angular: {z: -1.5}
+      <output type="ignition.msgs.Twist" topic="/keyboard_cmd">
+        linear: {x: 0.0}, angular: {z: -2.5}
       </output>
     </plugin>
@@ -70,5 +70,5 @@
         <match field="data">83</match>
       </input>
-      <output type="ignition.msgs.Twist" topic="/cmd_vel">
+      <output type="ignition.msgs.Twist" topic="/keyboard_cmd">
         linear: {x: 0.0}, angular: {z: 0.0}
       </output>
@@ -81,5 +81,5 @@
       <pose>0 0 0 0 0 0</pose>
       <topic>lidar</topic>
-      <update_rate>10</update_rate>
+      <update_rate>5</update_rate>
       <ray>
         <scan>
@@ -87,6 +87,6 @@
             <samples>640</samples>
             <resolution>1</resolution>
-            <min_angle>-1.396263</min_angle>  <!-- ~-80° -->
-            <max_angle>1.396263</max_angle>    <!-- ~80° -->
+            <min_angle>${-PI}</min_angle>
+            <max_angle>${PI}</max_angle>
           </horizontal>
           <vertical>
@@ -108,4 +108,39 @@
           name="ignition::gazebo::systems::Sensors">
         <render_engine>ogre2</render_engine>
+      </plugin>
+      <plugin filename="libignition-gazebo-joint-controller-system.so"
+          name="ignition::gazebo::systems::JointController">
+        <joint_name>rod_to_lidar</joint_name>
+        <use_velocity_control>false</use_velocity_control>
+        <use_position_control>true</use_position_control>
+      </plugin>
+    </sensor>
+  </gazebo>
+  <!-- Camera Plugins -->
+  <gazebo reference="camera_link">
+    <sensor name="camera_sensor" type="camera">
+      <pose>0 0 0 0 0 0</pose>  <!-- Adjust if camera is offset -->
+      <camera>
+        <horizontal_fov>1.047</horizontal_fov>  <!-- 60° FOV -->
+        <image>
+          <width>640</width>
+          <height>480</height>
+          <format>R8G8B8</format>
+        </image>
+        <clip>
+          <near>0.1</near>
+          <far>100</far>
+        </clip>
+      </camera>
+      <always_on>true</always_on>
+      <update_rate>30</update_rate>
+      <visualize>true</visualize>
+      <topic>camera/image_raw</topic>  <!-- ROS 2 topic -->
+      <plugin filename="libignition-gazebo-camera-system.so"
+              name="ignition::gazebo::systems::Camera">
+        <ros>
+          <namespace>/</namespace>
+          <remapping>~/image_raw:=camera/image_raw</remapping>
+        </ros>
       </plugin>
     </sensor>

File: src/simple_box_robo/model/robot.urdf.xacro (robot description, xacro)
@@ -244,10 +244,8 @@
     </inertial>
   </link>
-  <joint name="rod_to_lidar" type="revolute">
+  <joint name="rod_to_lidar" type="fixed">
     <parent link="rod" />
     <child link="lidar_body" />
     <origin xyz="0 0 ${rod_z/2 - lidar_z/4}" rpy="0 0 0" />
-    <axis xyz="0 0 1" />
-    <limit lower="${-3*PI/4}" upper="${3*PI/4}" effort="10.0" velocity="1.0" />
   </joint>
   <!-- Camera sensor -->
